File: pcb/adatv2.kicad_pcb (KiCad board)
At the start: 4 copper layers, 371.6 x 208.9 mm, 231 parts, among them J101 TO_IO, J102 TO_DISP_INPUT, J103 TO_DISP_OUTPUT, J104 WORD_CLK_1, J105 USB_C_Receptacle_USB2.0_14P, J106 WORD_CLK_2, J107 WORD_CLK_3, J108 WORD_CLK_4, J109 FPGA_JTAG, J110 STDC14_SWD, J201 9-15V DC, J202 PLR237, J203 PLT237, J204 PLT237, J205 TO_MAIN, J206 PLR237, J207 PLT237, J208 PLT237, J301 TO_MAIN, SW301 SAMPLE RATE, SW302 LOOPBACK, U101 10M02SCE144, U102 74LVC2G17, U103 74LVC2G17, U104 74LVC2G17, U105 74LVC2G17, U106 USB3300-EZK, U107 STM32F427VGTx, U201 AMS1117-3.3, U202 TPS56124x, U301 HT1635D, Y101 24.000MHz, Y102 OT2EL89CJI-111YLC-11.2896M, Y103 ECS-TXO-3225MV-122.8-TR

Commit message: Start routing main board
Parts:
- added C151: 100n, Capacitor_SMD:C_0805_2012Metric_Pad1.18x1.45mm_HandSolder, F.Cu at (230.9, 214.4)
- added C152: 100n, Capacitor_SMD:C_0805_2012Metric_Pad1.18x1.45mm_HandSolder, F.Cu at (225.8, 216.3)
- added C153: 100n, Capacitor_SMD:C_0805_2012Metric_Pad1.18x1.45mm_HandSolder, F.Cu at (225.3, 205.2)
- added C154: 100n, Capacitor_SMD:C_0805_2012Metric_Pad1.18x1.45mm_HandSolder, B.Cu at (229.9, 194.1)
- added C155: 100n, Capacitor_SMD:C_0805_2012Metric_Pad1.18x1.45mm_HandSolder, F.Cu at (154.9, 72.9)
- added C156: 100n, Capacitor_SMD:C_0805_2012Metric_Pad1.18x1.45mm_HandSolder, F.Cu at (154.9, 75.9)
- C101, C102, C103, C104, C105, C106, C107, C108, C109, C110, C111, C112, C113, C114, C115, C116, C117, C118, C121, C122, C123, C124, C125, C126, C127, C128, C134, C135, C136, C140, C141, L101: moved to B.Cu
- moved H102 308.3 mm to (294.0, 233.0)
- moved J109 270.8 mm to (292.1, 203.2)
- moved H104 265.3 mm to (294.0, 156.0)
- moved R129 261.9 mm to (285.0, 222.5), turned to -90 degrees
- moved R130 255.2 mm to (278.9, 222.5), turned to -90 degrees
- moved J108 254.2 mm to (282.0, 231.0), turned to 180 degrees
- moved R127 252.2 mm to (269.0, 222.5), turned to -90 degrees
- moved J107 251.3 mm to (266.0, 231.0), turned to 180 degrees
- moved J106 248.3 mm to (250.0, 231.0), turned to 180 degrees
- moved H101 248.1 mm to (206.0, 233.0)
- moved R128 245.5 mm to (262.9, 222.5), turned to -90 degrees
- moved J104 245.4 mm to (234.0, 231.0), turned to 180 degrees
- moved D107 240.9 mm to (274.1, 229.9)
- moved R125 236.1 mm to (253.0, 222.5), turned to -90 degrees
- moved R121 230.8 mm to (237.0, 222.5), turned to -90 degrees
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Routing:
- net WORD_CLK: track 0.00 -> 58.6 mm
- net /MCU and USB/MCO1: track 0.00 -> 55.2 mm, vias 0 -> 2
- net /MCU and USB/ULPI_D0: track 0.00 -> 41.8 mm
- net /MCU and USB/ULPI_D3: track 0.00 -> 41.7 mm
- net /MCU and USB/ULPI_D5: track 0.00 -> 41.7 mm
- net /MCU and USB/ULPI_D6: track 0.00 -> 41.6 mm
- net /MCU and USB/ULPI_D2: track 0.00 -> 41.4 mm
- net /MCU and USB/ULPI_NXT: track 0.00 -> 40.7 mm, vias 0 -> 2
- net /MCU and USB/ULPI_D1: track 0.00 -> 40.4 mm
- net /MCU and USB/ULPI_D4: track 0.00 -> 40.2 mm
- net /MCU and USB/ULPI_D7: track 0.00 -> 40.2 mm, vias 0 -> 2
- net /MCU and USB/ULPI_DIR: track 0.00 -> 38.7 mm, vias 0 -> 2
- net /MCU and USB/ULPI_CLK: track 0.00 -> 38.7 mm, vias 0 -> 2
- net /MCU and USB/ULPI_STP: track 0.00 -> 37.4 mm, vias 0 -> 2
- net /MCU and USB/USB_RESET: track 0.00 -> 29.1 mm, vias 0 -> 2
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Other:
- board size 371.6 x 208.9 mm -> 371.6 x 209 mm
- board text added: "+3V3"
- board text removed: "+3V"
