File: pcb/production/main-board.kicad_pcb (KiCad board)
At the start: 4 copper layers, 100 x 74 mm, 152 parts, among them J101 TO_IO, J102 TO_DISP_INPUT, J103 TO_DISP_OUTPUT, J104 WORD_CLK_1, J105 USB_C_Receptacle_USB2.0_14P, J106 WORD_CLK_2, J107 WORD_CLK_3, J108 WORD_CLK_4, J109 FPGA_JTAG, J110 STDC14_SWD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

Commit message: Provide final rev 1.0a production files
Parts:
- moved C111 35.8 mm to (101.9, 43.2)
- moved C112 35.8 mm to (101.9, 47.2)
- moved C113 35.8 mm to (101.9, 51.1)
- moved C115 35.8 mm to (95.5, 59.4)
- moved C118 35.8 mm to (47.1, 59.4)
- moved C145 35.8 mm to (98.2, 71.1)
- moved C148 35.8 mm to (98.5, 63.5)
- moved C157 35.8 mm to (63.9, 49.9)
- moved R130 35.8 mm to (99.3, 82.3)
- moved TP104 35.8 mm to (102.3, 34.8)
- moved TP107 35.8 mm to (115.5, 39.7)
- moved TP108 35.8 mm to (98.9, 33.0)
- moved U105 35.8 mm to (102.3, 77.9)
- moved C101 35.8 mm to (85.3, 59.4)
- moved C104 35.8 mm to (85.3, 53.2)
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Routing:
- net ADAT_OUT2_USER3: track 38.3 -> 39.4 mm
- net GND: track 192.5 -> 193.4 mm, vias 113 -> 120
- net Net-(U107-VCAP_2): track 5.31 -> 4.74 mm
